Commit message: Added panda gripper

File: urdf/go2_z1_description.urdf (robot description, URDF)
Before this commit: robot go2_z1_description, 37 links, 36 joints
Links:
- added link panda_hand, mass 0.73; collision mesh filename=../meshes/panda_collision/hand.stl scale=1 0.6 1; visual mesh filename=../meshes/panda_visual/hand.dae scale=1 0.6 1
- added link panda_hand_tcp
- added link panda_leftfinger, mass 0.015; collision box size=17.5e-3 15.2e-3 18.5e-3; collision box size=17.5e-3 7e-3 23.5e-3
- added link panda_leftfinger_pad
- added link panda_link7, mass 0.735522; collision mesh filename=../meshes/panda_collision/link7.stl; visual mesh filename=../meshes/panda_visual/link7.dae
- added link panda_link8
- added link panda_rightfinger, mass 0.015; collision box size=17.5e-3 15.2e-3 18.5e-3; collision box size=17.5e-3 7e-3 23.5e-3
- added link panda_rightfinger_pad
Joints:
- added joint panda_finger_joint1: type prismatic, parent panda_hand, child panda_leftfinger, origin xyz=0 0 0.0584 rpy=0 0 0, axis 0 1 0, limit lower=0.0 upper=0.04 effort=100 velocity=0.2
- added joint panda_finger_joint2: type prismatic, parent panda_hand, child panda_rightfinger, origin xyz=0 0 0.0584 rpy=0 0 0, axis 0 -1 0, limit lower=0.0 upper=0.04 effort=100 velocity=0.2, mimic joint=panda_finger_joint1
- added joint panda_hand_joint: type fixed, parent panda_link8, child panda_hand, origin xyz=0 0 0 rpy=0 0 -0.7853981633974483
- added joint panda_hand_tcp_joint: type fixed, parent panda_hand, child panda_hand_tcp, origin xyz=0 0 0.1034 rpy=0 0 0
- added joint panda_joint7: type fixed, parent z1_link06, child panda_link7, origin xyz=0 0 0 rpy=0 1.570796 0, axis 0 0 1, limit lower=-2.8973 upper=2.8973 effort=12 velocity=2.6100
- added joint panda_joint8: type fixed, parent panda_link7, child panda_link8, origin xyz=0 0 0.107 rpy=0 0 0
- added joint panda_leftfinger_pad_joint: type fixed, parent panda_leftfinger, child panda_leftfinger_pad, origin xyz=0 0 0.0455 rpy=0 0 0
- added joint panda_rightfinger_pad_joint: type fixed, parent panda_rightfinger, child panda_rightfinger_pad, origin xyz=0 0 0.0455 rpy=0 0 0
- joint go2_z1_joint: origin xyz=0 0 0.057 rpy=0 0 0 -> xyz=0.13 0 0.06 rpy=0 0 0
